File: kicad/PS400-5/PS400-4.sch (KiCad schematic (older format))
At the start: 28 parts, among them J1 Conn, J2 Conn, J3 Conn, J4 Conn, J5 Conn, Q1 RUM002N05, Q2 Q_NPN_BEC, Q3 RUM002N05, T1 B82801A150, U2 PIC10F206-IOT

Commit message: изменено:      Documents/circuit.png 	изменено:      kicad/PS400-5/PS400-4.kicad_pcb 	изменено:      kicad/PS400-5/PS400-4.kicad_pcb-bak 	изменено:      kicad/PS400-5/PS400-4.pdf 	изменено:      kicad/PS400-5/PS400-4.sch 	изменено:      kicad/PS400-5/PS400-4.sch-bak
Connections:
- net at U2.3 (GP1): now also Q3.1 (G), R8.2; no longer Q2.3 (C)
- new net: Q2.3 (C), U2.6 (GP3)
Other:
- moved on the sheet: C2, J4, J5, Q2, Q3, R7, R8
Changed lines of the file:
@@
 L Device:Q_NPN_BEC Q2
 U 1 1 624E03F2
-P 5650 3850
-F 0 "Q2" H 5841 3896 50  0000 L CNN
-F 1 "Q_NPN_BEC" H 5841 3805 50  0000 L CNN
-F 2 "Package_TO_SOT_SMD:SOT-23" H 5850 3950 50  0001 C CNN
-F 3 "~" H 5650 3850 50  0001 C CNN
-	1    5650 3850
+P 6900 3900
+F 0 "Q2" H 7091 3946 50  0000 L CNN
+F 1 "Q_NPN_BEC" H 7091 3855 50  0000 L CNN
+F 2 "Package_TO_SOT_SMD:SOT-23" H 7100 4000 50  0001 C CNN
+F 3 "~" H 6900 3900 50  0001 C CNN
+	1    6900 3900
 	1    0    0    -1
 $EndComp
@@
 L Device:R R7
 U 1 1 624E0B44
-P 5450 4000
-F 0 "R7" H 5350 4000 50  0000 R CNN
-F 1 "10k" H 5350 4100 50  0000 R CNN
-F 2 "Resistor_SMD:R_0402_1005Metric" V 5380 4000 50  0001 C CNN
-F 3 "~" H 5450 4000 50  0001 C CNN
-	1    5450 4000
+P 6700 4050
+F 0 "R7" H 6600 4050 50  0000 R CNN
+F 1 "10k" H 6600 4150 50  0000 R CNN
+F 2 "Resistor_SMD:R_0402_1005Metric" V 6630 4050 50  0001 C CNN
+F 3 "~" H 6700 4050 50  0001 C CNN
+	1    6700 4050
 	-1   0    0    1
 $EndComp
@@
 L Device:C C2
 U 1 1 624E12F8
-P 5300 4000
-F 0 "C2" H 5000 4000 50  0000 L CNN
-F 1 "100" H 5000 3900 50  0000 L CNN
-F 2 "Capacitor_SMD:C_0402_1005Metric" H 5338 3850 50  0001 C CNN
-F 3 "~" H 5300 4000 50  0001 C CNN
-	1    5300 4000
+P 6550 4050
+F 0 "C2" H 6250 4050 50  0000 L CNN
+F 1 "100" H 6250 3950 50  0000 L CNN
+F 2 "Capacitor_SMD:C_0402_1005Metric" H 6588 3900 50  0001 C CNN
+F 3 "~" H 6550 4050 50  0001 C CNN
+	1    6550 4050
 	1    0    0    -1
 $EndComp
@@
 L power:GND #PWR02
 U 1 1 624E1A68
-P 5750 4150
-F 0 "#PWR02" H 5750 3900 50  0001 C CNN
-F 1 "GND" H 5755 3977 50  0001 C CNN
-F 2 "" H 5750 4150 50  0001 C CNN
-F 3 "" H 5750 4150 50  0001 C CNN
-	1    5750 4150
+P 7000 4200
+F 0 "#PWR02" H 7000 3950 50  0001 C CNN
+F 1 "GND" H 7005 4027 50  0001 C CNN
+F 2 "" H 7000 4200 50  0001 C CNN
+F 3 "" H 7000 4200 50  0001 C CNN
+	1    7000 4200
 	1    0    0    -1
 $EndComp
 Wire Wire Line
-	5750 4150 5750 4050
-Connection ~ 5750 4150
-Connection ~ 5450 4150
+	7000 4200 7000 4100
+Connection ~ 7000 4200
+Connection ~ 6700 4200
 Wire Wire Line
-	5450 4150 5750 4150
+	6700 4200 7000 4200
 Wire Wire Line
-	5300 3850 5450 3850
+	6550 3900 6700 3900
 Wire Wire Line
-	5300 4150 5450 4150
-Connection ~ 5450 3850
+	6550 4200 6700 4200
+Connection ~ 6700 3900
 $Comp
 L PS400-4-rescue:Conn-My_Library J4
 U 1 1 624E7EDC
-P 5100 3850
-F 0 "J4" H 5042 3757 50  0000 C CNN
-F 1 "Conn" H 5042 3756 50  0001 C CNN
-F 2 "My-library:SMD-CONN" H 5150 3700 50  0001 C CNN
-F 3 "~" H 5100 3850 50  0001 C CNN
-	1    5100 3850
+P 6350 3900
+F 0 "J4" H 6292 3807 50  0000 C CNN
+F 1 "Conn" H 6292 3806 50  0001 C CNN
+F 2 "My-library:SMD-CONN" H 6400 3750 50  0001 C CNN
+F 3 "~" H 6350 3900 50  0001 C CNN
+	1    6350 3900
 	-1   0    0    1
 $EndComp
 Wire Wire Line
-	5200 3850 5300 3850
-Connection ~ 5300 3850
+	6450 3900 6550 3900
+Connection ~ 6550 3900
 Wire Wire Line
 	7200 3250 7500 3250
@@
 L Device:Q_NMOS_GSD Q3
 U 1 1 624FC070
-P 7200 3850
-F 0 "Q3" H 7406 3896 50  0000 L CNN
-F 1 "RUM002N05" H 7406 3805 50  0000 L CNN
-F 2 "Package_TO_SOT_SMD:SOT-723" H 7400 3950 50  0001 C CNN
-F 3 "~" H 7200 3850 50  0001 C CNN
-	1    7200 3850
+P 5950 3900
+F 0 "Q3" H 5450 4150 50  0000 L CNN
+F 1 "RUM002N05" H 5200 4050 50  0000 L CNN
+F 2 "Package_TO_SOT_SMD:SOT-723" H 6150 4000 50  0001 C CNN
+F 3 "~" H 5950 3900 50  0001 C CNN
+	1    5950 3900
 	1    0    0    -1
 $EndComp
@@
 L power:GND #PWR03
 U 1 1 624FD7EC
-P 7300 4150
-F 0 "#PWR03" H 7300 3900 50  0001 C CNN
-F 1 "GND" H 7305 3977 50  0001 C CNN
-F 2 "" H 7300 4150 50  0001 C CNN
-F 3 "" H 7300 4150 50  0001 C CNN
-	1    7300 4150
+P 6050 4200
+F 0 "#PWR03" H 6050 3950 50  0001 C CNN
+F 1 "GND" H 6055 4027 50  0001 C CNN
+F 2 "" H 6050 4200 50  0001 C CNN
+F 3 "" H 6050 4200 50  0001 C CNN
+	1    6050 4200
 	1    0    0    -1
 $EndComp
@@
 L PS400-4-rescue:Conn-My_Library J5
 U 1 1 624FDF1C
-P 7400 3650
-F 0 "J5" H 7500 3650 50  0000 C CNN
-F 1 "Conn" H 7342 3556 50  0001 C CNN
-F 2 "My-library:SMD-CONN" H 7450 3500 50  0001 C CNN
-F 3 "~" H 7400 3650 50  0001 C CNN
-	1    7400 3650
+P 6150 3700
+F 0 "J5" H 6250 3700 50  0000 C CNN
+F 1 "Conn" H 6092 3606 50  0001 C CNN
+F 2 "My-library:SMD-CONN" H 6200 3550 50  0001 C CNN
+F 3 "~" H 6150 3700 50  0001 C CNN
+	1    6150 3700
 	1    0    0    -1
 $EndComp
@@
 L Device:R R8
 U 1 1 624FE8AB
-P 7000 4000
-F 0 "R8" H 7250 3950 50  0000 R CNN
-F 1 "100k" H 7300 4050 50  0000 R CNN
-F 2 "Resistor_SMD:R_0402_1005Metric" V 6930 4000 50  0001 C CNN
-F 3 "~" H 7000 4000 50  0001 C CNN
-	1    7000 4000
+P 5750 4050
+F 0 "R8" H 6000 4000 50  0000 R CNN
+F 1 "100k" H 6050 4100 50  0000 R CNN
+F 2 "Resistor_SMD:R_0402_1005Metric" V 5680 4050 50  0001 C CNN
+F 3 "~" H 5750 4050 50  0001 C CNN
+	1    5750 4050
 	-1   0    0    1
 $EndComp
 Wire Wire Line
-	7000 4150 7300 4150
+	5750 4200 6050 4200
 Wire Wire Line
-	7300 4150 7300 4050
-Connection ~ 7300 4150
+	6050 4200 6050 4100
+Connection ~ 6050 4200
 Wire Wire Line
 	6950 2750 7000 2750
@@
 	5300 2750 5500 2750
 Wire Wire Line
-	5750 2950 5750 3650
+	7000 2750 7000 3700
 Wire Wire Line
-	7000 2750 7000 3850
-Connection ~ 7000 3850
+	5750 2950 5750 3900
+Connection ~ 5750 3900
 $EndSCHEMATC

Commit message: изменено:      Documents/circuit.png 	изменено:      kicad/PS400-5/PS400-4-cache.lib 	изменено:      kicad/PS400-5/PS400-4.kicad_pcb 	изменено:      kicad/PS400-5/PS400-4.kicad_pcb-bak 	изменено:      kicad/PS400-5/PS400-4.pdf 	изменено:      kicad/PS400-5/PS400-4.sch 	изменено:      kicad/PS400-5/PS400-4.sch-bak
Parts:
- removed J5: Conn, My-library:SMD-CONN, symbol PS400-4-rescue:Conn-My_Library
- added BZ1: Buzzer, My-library:BuzerSMD, symbol Device:Buzzer
- C2: value 100 -> 200
- J1: value Conn -> +BAT
- J2: value Conn -> +GM
- J3: value Conn -> -BAT
- J4: value Conn -> -GM
Connections:
- net +3V3: now also BZ1.1 (-)
- net at Q3.3 (D): now also BZ1.2 (+)
Other:
- moved on the sheet: C2, Q2, R7
Changed lines of the file:
@@
 U 1 1 61859C20
 P 6350 2850
-F 0 "U2" H 6350 2850 50  0000 C CNN
-F 1 "PIC10F206-IOT" H 6350 3050 50  0000 C CNN
+F 0 "U2" H 6350 2950 50  0000 C CNN
+F 1 "PIC10F206-IOT" H 6350 2850 50  0000 C CNN
 F 2 "Package_TO_SOT_SMD:SOT-23-6" H 6400 3500 50  0001 L CIN
 F 3 "http://ww1.microchip.com/downloads/en/DeviceDoc/41239D.pdf" H 6350 2850 50  0001 C CNN
@@
 U 1 1 6185A482
 P 6600 2150
-F 0 "R1" V 6393 2150 50  0000 C CNN
-F 1 "47" V 6484 2150 50  0000 C CNN
+F 0 "R1" V 6400 2150 50  0000 C CNN
+F 1 "47" V 6500 2150 50  0000 C CNN
 F 2 "Resistor_SMD:R_0402_1005Metric" V 6530 2150 50  0001 C CNN
 F 3 "~" H 6600 2150 50  0001 C CNN
@@
 U 1 1 6185A86F
 P 7300 2450
-F 0 "T1" H 7300 2975 50  0000 C CNN
-F 1 "B82801A150" H 7400 2900 50  0000 C CNN
+F 0 "T1" H 7400 2950 50  0000 C CNN
+F 1 "B82801A150" H 7400 2850 50  0000 C CNN
 F 2 "My-library:B82801A1" H 7300 2450 50  0001 C CNN
 F 3 "" H 7300 2450 50  0001 C CNN
@@
 U 1 1 6185B1E9
 P 7400 2950
-F 0 "Q1" H 7250 3250 50  0000 L CNN
-F 1 "RUM002N05" H 7050 3150 50  0000 L CNN
+F 0 "Q1" H 7200 3350 50  0000 L CNN
+F 1 "RUM002N05" H 7000 3250 50  0000 L CNN
 F 2 "Package_TO_SOT_SMD:SOT-723" H 7600 3050 50  0001 C CNN
 F 3 "~" H 7400 2950 50  0001 C CNN
@@
 $EndComp
 $Comp
-L power:+3.3V #PWR01
-U 1 1 6185CB16
-P 5800 2150
-F 0 "#PWR01" H 5800 2000 50  0001 C CNN
-F 1 "+3.3V" H 5815 2323 50  0000 C CNN
-F 2 "" H 5800 2150 50  0001 C CNN
-F 3 "" H 5800 2150 50  0001 C CNN
-	1    5800 2150
-	1    0    0    -1
-$EndComp
-$Comp
 L Device:D D2
 U 1 1 6186223A
@@
 U 1 1 61862636
 P 8450 2150
-F 0 "D3" H 8450 1934 50  0000 C CNN
-F 1 "RS1JL" H 8450 2025 50  0000 C CNN
+F 0 "D3" H 8450 1950 50  0000 C CNN
+F 1 "RS1JL" H 8450 2050 50  0000 C CNN
 F 2 "Diode_SMD:D_SOD-123" H 8450 2150 50  0001 C CNN
 F 3 "~" H 8450 2150 50  0001 C CNN
@@
 U 1 1 6186558C
 P 7900 1950
-F 0 "C1" V 7800 1850 50  0000 C CNN
-F 1 "10n" V 7800 2100 50  0000 C CNN
+F 0 "C1" V 7850 1800 50  0000 C CNN
+F 1 "10n" V 7850 2100 50  0000 C CNN
 F 2 "Capacitor_SMD:C_1812_4532Metric" H 7938 1800 50  0001 C CNN
 F 3 "~" H 7900 1950 50  0001 C CNN
@@
 	-1   0    0    1
 $EndComp
-Connection ~ 5800 2150
 Wire Wire Line
 	5800 2150 6350 2150
 Wire Wire Line
 	6350 2250 6350 2150
-Wire Wire Line
-	7500 2550 7500 2400
 Wire Wire Line
 	7800 2150 8000 2150
@@
 L PS400-4-rescue:Conn-My_Library J1
 U 1 1 6189986E
-P 4950 2150
-F 0 "J1" H 4892 2057 50  0000 C CNN
-F 1 "Conn" H 4892 2056 50  0001 C CNN
-F 2 "My-library:SMD-CONN" H 5000 2000 50  0001 C CNN
-F 3 "~" H 4950 2150 50  0001 C CNN
-	1    4950 2150
+P 5250 2150
+F 0 "J1" H 5192 2057 50  0001 C CNN
+F 1 "+BAT" H 5200 2100 50  0000 C CNN
+F 2 "My-library:SMD-CONN" H 5300 2000 50  0001 C CNN
+F 3 "~" H 5250 2150 50  0001 C CNN
+	1    5250 2150
 	-1   0    0    1
 $EndComp
@@
 U 1 1 6189AD72
 P 8750 2150
-F 0 "R2" V 8543 2150 50  0000 C CNN
-F 1 "4.7M" V 8634 2150 50  0000 C CNN
+F 0 "R2" V 8550 2150 50  0000 C CNN
+F 1 "4.7M" V 8650 2150 50  0000 C CNN
 F 2 "Resistor_SMD:R_0603_1608Metric" V 8680 2150 50  0001 C CNN
 F 3 "~" H 8750 2150 50  0001 C CNN
@@
 U 1 1 6189B2E9
 P 9300 2150
-F 0 "J2" H 9328 2150 50  0000 L CNN
-F 1 "Conn" H 9242 2056 50  0001 C CNN
+F 0 "J2" H 9328 2150 50  0001 L CNN
+F 1 "+GM" H 9250 2250 50  0000 C CNN
 F 2 "My-library:SMD-CONN" H 9350 2000 50  0001 C CNN
 F 3 "~" H 9300 2150 50  0001 C CNN
@@
 U 1 1 6189B7D6
 P 9050 2150
-F 0 "R3" V 8843 2150 50  0000 C CNN
-F 1 "4.7M" V 8934 2150 50  0000 C CNN
+F 0 "R3" V 8850 2150 50  0000 C CNN
+F 1 "4.7M" V 8950 2150 50  0000 C CNN
 F 2 "Resistor_SMD:R_0603_1608Metric" V 8980 2150 50  0001 C CNN
 F 3 "~" H 9050 2150 50  0001 C CNN
@@
 L PS400-4-rescue:Conn-My_Library J3
 U 1 1 61B9B598
-P 4900 3350
-F 0 "J3" H 4842 3257 50  0000 C CNN
-F 1 "Conn" H 4842 3256 50  0001 C CNN
-F 2 "My-library:SMD-CONN" H 4950 3200 50  0001 C CNN
-F 3 "~" H 4900 3350 50  0001 C CNN
-	1    4900 3350
+P 5250 2450
+F 0 "J3" H 5192 2357 50  0001 C CNN
+F 1 "-BAT" H 5200 2400 50  0000 C CNN
+F 2 "My-library:SMD-CONN" H 5300 2300 50  0001 C CNN
+F 3 "~" H 5250 2450 50  0001 C CNN
+	1    5250 2450
 	-1   0    0    1
 $EndComp
@@
 L power:GND #PWR011
 U 1 1 61B9BC32
-P 5000 3350
-F 0 "#PWR011" H 5000 3100 50  0001 C CNN
-F 1 "GND" H 5005 3177 50  0001 C CNN
-F 2 "" H 5000 3350 50  0001 C CNN
-F 3 "" H 5000 3350 50  0001 C CNN
-	1    5000 3350
+P 5350 2450
+F 0 "#PWR011" H 5350 2200 50  0001 C CNN
+F 1 "GND" H 5355 2277 50  0001 C CNN
+F 2 "" H 5350 2450 50  0001 C CNN
+F 3 "" H 5350 2450 50  0001 C CNN
+	1    5350 2450
 	1    0    0    -1
 $EndComp
@@
 	1    0    0    -1
 $EndComp
-Wire Wire Line
-	5050 2150 5800 2150
 $Comp
 L Device:Q_NPN_BEC Q2
 U 1 1 624E03F2
-P 6900 3900
-F 0 "Q2" H 7091 3946 50  0000 L CNN
-F 1 "Q_NPN_BEC" H 7091 3855 50  0000 L CNN
-F 2 "Package_TO_SOT_SMD:SOT-23" H 7100 4000 50  0001 C CNN
-F 3 "~" H 6900 3900 50  0001 C CNN
-	1    6900 3900
-	1    0    0    -1
+P 7100 3900
+F 0 "Q2" H 6950 4050 50  0000 L CNN
+F 1 "Q_NPN_BEC" H 7291 3855 50  0001 L CNN
+F 2 "Package_TO_SOT_SMD:SOT-23" H 7300 4000 50  0001 C CNN
+F 3 "~" H 7100 3900 50  0001 C CNN
+	1    7100 3900
+	-1   0    0    -1
 $EndComp
 $Comp
 L Device:R R7
 U 1 1 624E0B44
-P 6700 4050
-F 0 "R7" H 6600 4050 50  0000 R CNN
-F 1 "10k" H 6600 4150 50  0000 R CNN
-F 2 "Resistor_SMD:R_0402_1005Metric" V 6630 4050 50  0001 C CNN
-F 3 "~" H 6700 4050 50  0001 C CNN
-	1    6700 4050
+P 7450 4050
+F 0 "R7" H 7350 4050 50  0000 R CNN
+F 1 "10k" H 7350 4150 50  0000 R CNN
+F 2 "Resistor_SMD:R_0402_1005Metric" V 7380 4050 50  0001 C CNN
+F 3 "~" H 7450 4050 50  0001 C CNN
+	1    7450 4050
 	-1   0    0    1
 $EndComp
@@
 L Device:C C2
 U 1 1 624E12F8
-P 6550 4050
-F 0 "C2" H 6250 4050 50  0000 L CNN
-F 1 "100" H 6250 3950 50  0000 L CNN
-F 2 "Capacitor_SMD:C_0402_1005Metric" H 6588 3900 50  0001 C CNN
-F 3 "~" H 6550 4050 50  0001 C CNN
-	1    6550 4050
+P 7300 4050
+F 0 "C2" H 7100 4050 50  0000 L CNN
+F 1 "200" H 7050 3950 50  0000 L CNN
+F 2 "Capacitor_SMD:C_0402_1005Metric" H 7338 3900 50  0001 C CNN
+F 3 "~" H 7300 4050 50  0001 C CNN
+	1    7300 4050
 	1    0    0    -1
 $EndComp
@@
 Wire Wire Line
 	7000 4200 7000 4100
-Connection ~ 7000 4200
-Connection ~ 6700 4200
-Wire Wire Line
-	6700 4200 7000 4200
-Wire Wire Line
-	6550 3900 6700 3900
-Wire Wire Line
-	6550 4200 6700 4200
-Connection ~ 6700 3900
 $Comp
 L PS400-4-rescue:Conn-My_Library J4
 U 1 1 624E7EDC
-P 6350 3900
-F 0 "J4" H 6292 3807 50  0000 C CNN
-F 1 "Conn" H 6292 3806 50  0001 C CNN
-F 2 "My-library:SMD-CONN" H 6400 3750 50  0001 C CNN
-F 3 "~" H 6350 3900 50  0001 C CNN
-	1    6350 3900
-	-1   0    0    1
-$EndComp
-Wire Wire Line
-	6450 3900 6550 3900
-Connection ~ 6550 3900
+P 7650 3900
+F 0 "J4" H 7592 3807 50  0001 C CNN
+F 1 "-GM" H 7650 4000 50  0000 C CNN
+F 2 "My-library:SMD-CONN" H 7700 3750 50  0001 C CNN
+F 3 "~" H 7650 3900 50  0001 C CNN
+	1    7650 3900
+	1    0    0    -1
+$EndComp
 Wire Wire Line
 	7200 3250 7500 3250
@@
 	7500 3250 7500 3150
 Connection ~ 7500 3250
-Wire Wire Line
-	7500 2550 7500 2750
-Connection ~ 7500 2550
 $Comp
 L Device:Q_NMOS_GSD Q3
@@
 $EndComp
 $Comp
-L PS400-4-rescue:Conn-My_Library J5
-U 1 1 624FDF1C
-P 6150 3700
-F 0 "J5" H 6250 3700 50  0000 C CNN
-F 1 "Conn" H 6092 3606 50  0001 C CNN
-F 2 "My-library:SMD-CONN" H 6200 3550 50  0001 C CNN
-F 3 "~" H 6150 3700 50  0001 C CNN
-	1    6150 3700
-	1    0    0    -1
-$EndComp
-$Comp
 L Device:R R8
 U 1 1 624FE8AB
@@
 Connection ~ 6350 2150
 Wire Wire Line
-	7100 2550 7500 2550
-Wire Wire Line
-	7100 2400 7100 2550
-Wire Wire Line
 	6950 2950 7200 2950
 Connection ~ 7200 2950
@@
 	5750 2950 5750 3900
 Connection ~ 5750 3900
+Wire Wire Line
+	5350 2150 5800 2150
+Connection ~ 5800 2150
+Wire Wire Line
+	7450 4200 7300 4200
+Connection ~ 7000 4200
+Connection ~ 7300 4200
+Wire Wire Line
+	7300 4200 7000 4200
+Wire Wire Line
+	7300 3900 7450 3900
+Connection ~ 7300 3900
+Connection ~ 7450 3900
+Wire Wire Line
+	7450 3900 7550 3900
+Wire Wire Line
+	7500 2400 7500 2500
+Wire Wire Line
+	7100 2400 7100 2500
+Wire Wire Line
+	7100 2500 7500 2500
+Connection ~ 7500 2500
+Wire Wire Line
+	7500 2500 7500 2750
+$Comp
+L Device:Buzzer BZ1
+U 1 1 62548A5C
+P 6400 3800
+F 0 "BZ1" H 6404 3475 50  0000 C CNN
+F 1 "Buzzer" H 6404 3566 50  0000 C CNN
+F 2 "My-library:BuzerSMD" V 6375 3900 50  0001 C CNN
+F 3 "~" V 6375 3900 50  0001 C CNN
+	1    6400 3800
+	1    0    0    1
+$EndComp
+Wire Wire Line
+	6050 3700 6300 3700
+$Comp
+L power:+3.3V #PWR0101
+U 1 1 6254C913
+P 6350 2150
+F 0 "#PWR0101" H 6350 2000 50  0001 C CNN
+F 1 "+3.3V" H 6365 2323 50  0000 C CNN
+F 2 "" H 6350 2150 50  0001 C CNN
+F 3 "" H 6350 2150 50  0001 C CNN
+	1    6350 2150
+	1    0    0    -1
+$EndComp
+$Comp
+L power:+3.3V #PWR0102
+U 1 1 6254DD6F
+P 6300 3900
+F 0 "#PWR0102" H 6300 3750 50  0001 C CNN
+F 1 "+3.3V" H 6315 4073 50  0000 C CNN
+F 2 "" H 6300 3900 50  0001 C CNN
+F 3 "" H 6300 3900 50  0001 C CNN
+	1    6300 3900
+	-1   0    0    1
+$EndComp
 $EndSCHEMATC
