File: kicad/PS400-5/PS400-4.kicad_pcb (KiCad board)
At the start: 2 copper layers, 13.5 x 13.1 mm, 28 parts, among them J1 Conn, J2 Conn, J3 Conn, J4 Conn, J5 Conn, Q1 RUM002N05, Q2 Q_NPN_BEC, Q3 RUM002N05, T1 B82801A150, U2 PIC10F206-IOT

Commit message: изменено:      Documents/circuit.png 	изменено:      kicad/PS400-5/PS400-4.kicad_pcb 	изменено:      kicad/PS400-5/PS400-4.kicad_pcb-bak 	изменено:      kicad/PS400-5/PS400-4.pdf 	изменено:      kicad/PS400-5/PS400-4.sch 	изменено:      kicad/PS400-5/PS400-4.sch-bak
Parts:
- moved C2 8.83 mm to (33.9, 49.4), turned to 180 degrees
- moved R7 7.70 mm to (33.9, 48.3), turned to 0 degrees
- moved J4 5.33 mm to (35.2, 46.9)
- moved J5 4.10 mm to (39.3, 48.0), turned to 270 degrees
- moved Q3 3.55 mm to (39.3, 50.1), turned to 90 degrees
- moved Q2 2.87 mm to (36.7, 49.3), turned to 0 degrees
- moved R8 2.59 mm to (39.3, 51.7), turned to 180 degrees
Connections:
- U2 pad 3: Net-(Q2-Pad3) -> Net-(Q3-Pad1)
- U2 pad 6: Net-(Q3-Pad1) -> Net-(Q2-Pad3)
Routing:
- net GND: track 21.4 -> 29.3 mm
- net Net-(Q3-Pad1): track 6.65 -> 2.51 mm
- net Net-(Q2-Pad3): track 3.76 -> 6.68 mm

Commit message: изменено:      Documents/circuit.png 	изменено:      kicad/PS400-5/PS400-4-cache.lib 	изменено:      kicad/PS400-5/PS400-4.kicad_pcb 	изменено:      kicad/PS400-5/PS400-4.kicad_pcb-bak 	изменено:      kicad/PS400-5/PS400-4.pdf 	изменено:      kicad/PS400-5/PS400-4.sch 	изменено:      kicad/PS400-5/PS400-4.sch-bak
Parts:
- removed J5: Conn, My-library:SMD-CONN
- added BZ1: Buzzer, My-library:BuzerSMD, F.Cu at (37.1, 49.1)
- C2: value 100 -> 200
- J1: value Conn -> +BAT
- J2: value Conn -> +GM
- J3: value Conn -> -BAT
- J4: value Conn -> -GM
- moved Q2 3.59 mm to (37.6, 45.8)
- moved C2 3.24 mm to (35.3, 46.5), turned to 270 degrees
- moved J4 2.07 mm to (34.8, 44.8)
- moved R7 1.91 mm to (34.3, 46.5), turned to 90 degrees
- moved R8 1.66 mm to (40.6, 52.8)
- moved Q3 1.50 mm to (39.4, 51.6), turned to 180 degrees
- moved R1 0.75 mm to (35.5, 51.3)
Routing:
- net Net-(Q2-Pad3): track 6.68 -> 10.4 mm
- net +3V3: track 5.21 -> 7.43 mm
- net GND: track 29.3 -> 30.7 mm
- net Net-(BZ1-Pad2): track 1.52 -> 2.67 mm
- net Net-(Q3-Pad1): track 2.51 -> 1.98 mm

Commit message: изменено:      kicad/PS400-5/PS400-4.kicad_pcb 	изменено:      kicad/PS400-5/PS400-4.kicad_pcb-bak 	изменено:      kicad/PS400-5/fp-info-cache
Parts:
- moved R7 9.26 mm to (43.5, 45.8), turned to 270 degrees
- moved J4 8.69 mm to (43.1, 47.5), turned to 180 degrees
- moved C2 7.18 mm to (42.5, 45.8), turned to 90 degrees
- moved Q2 2.96 mm to (40.6, 46.1), turned to 180 degrees
Routing:
- net GND: track 30.7 -> 18.6 mm
- net Net-(Q2-Pad3): track 10.4 -> 11.3 mm
